Commit message: update urdf.xacro and include the sim_biotec lib, not compiled successfully yet

File: sim_biotac_motorhand/robots/sim_biotac_motorhand_1.urdf.xacro (robot description, xacro)
@@ -1,4 +1,4 @@
 <?xml version="1.0"?>
-<robot
+<!--<robot
     xmlns:sensor="http://playerstage.sourceforge.net/gazebo/xmlschema/#sensor"
     xmlns:controller="http://playerstage.sourceforge.net/gazebo/xmlschema/#controller"
@@ -21,3 +21,69 @@
         </plugin>
     </gazebo>
+</robot>-->
+<!--
+ Software License Agreement (BSD License)
+ Copyright © 2022 belongs to Shadow Robot Company Ltd.
+ All rights reserved.
+ Redistribution and use in source and binary forms, with or without modification,
+ are permitted provided that the following conditions are met:
+   1. Redistributions of source code must retain the above copyright notice,
+      this list of conditions and the following disclaimer.
+   2. Redistributions in binary form must reproduce the above copyright notice,
+      this list of conditions and the following disclaimer in the documentation
+      and/or other materials provided with the distribution.
+   3. Neither the name of Shadow Robot Company Ltd nor the names of its contributors
+      may be used to endorse or promote products derived from this software without
+      specific prior written permission.
+ This software is provided by Shadow Robot Company Ltd "as is" and any express
+ or implied warranties, including, but not limited to, the implied warranties of
+ merchantability and fitness for a particular purpose are disclaimed. In no event
+ shall the copyright holder be liable for any direct, indirect, incidental, special,
+ exemplary, or consequential damages (including, but not limited to, procurement of
+ substitute goods or services; loss of use, data, or profits; or business interruption)
+ however caused and on any theory of liability, whether in contract, strict liability,
+ or tort (including negligence or otherwise) arising in any way out of the use of this
+ software, even if advised of the possibility of such damage.
+-->
+<robot xmlns:xacro="http://www.ros.org/wiki/xacro"
+       xmlns:sensor="http://playerstage.sourceforge.net/gazebo/xmlschema/#sensor"
+       xmlns:controller="http://playerstage.sourceforge.net/gazebo/xmlschema/#controller"
+       xmlns:interface="http://playerstage.sourceforge.net/gazebo/xmlschema/#interface"
+       name="shadowhand_motor">
+  <xacro:include filename="$(find sr_description)/other/xacro/materials.urdf.xacro"/>
+  <xacro:include filename="$(find sr_description)/hand/xacro/hand.urdf.xacro"/>
+  <xacro:include filename="$(find sr_description)/other/xacro/gazebo.urdf.xacro"/>
+  <xacro:arg name="hand_type" default="hand_e"/>
+  <xacro:arg name="hand_version" default="E3M5"/>
+  <xacro:arg name="side" default="right"/>
+  <xacro:arg name="fingers" default="all"/>
+  <xacro:arg name="tip_sensors" default="pst"/>
+  <xacro:arg name="mid_sensors" default="none"/>
+  <xacro:arg name="prox_sensors" default="none"/>
+  <xacro:arg name="palm_sensor" default="none"/>
+  <xacro:arg name="mounting_plate" default="false"/>
+  <link name="world" />
+  <xacro:if value="${'$(arg side)' == 'right'}">
+    <joint name="rh_world_joint" type="fixed">
+      <parent link="world" />
+      <child link="rh_forearm" />
+      <origin xyz="0.0 0.0 0.0" rpy="0.0 0.0 0.0" />
+    </joint>
+  </xacro:if>
+  <xacro:if value="${'$(arg side)' == 'left'}">
+    <joint name="lh_world_joint" type="fixed">
+      <parent link="world" />
+      <child link="lh_forearm" />
+      <origin xyz="0.0 0.0 0.0" rpy="0.0 0.0 0.0" />
+    </joint>
+  </xacro:if>
+  <xacro:sr_hand hand_type="$(arg hand_type)" hand_version="$(arg hand_version)" side="$(arg side)"
+                 fingers="$(arg fingers)" tip_sensors="$(arg tip_sensors)" mid_sensors="$(arg mid_sensors)"
+                 prox_sensors="$(arg prox_sensors)" palm_sensor="$(arg palm_sensor)" mounting_plate="$(arg mounting_plate)"/>
+    <gazebo>
+        <plugin filename="libsim_biotac.so" name="sim_biotac">
+            <alwaysOn>true</alwaysOn>
+            <updateRate>100.0</updateRate>
+        </plugin>
+    </gazebo>
 </robot>
